File: docs/PCB/BleRDF_receiver/BleRDF_receiver.kicad_sch (KiCad schematic)
At the start: 17 parts, among them J1 Conn_01x02, J2 Conn_01x02, J3 Conn_01x02, J5 Conn_01x09_Pin, SW2 SW_Push, SW3 SW_SPDT_312, U1 XIAO-ESP32-C6

Commit message: Update PCB wiring and add 3D case models
Connections:
- net GND: now also J3.2 (Pin_2), SW2.1
- net VCC: no longer J3.2 (Pin_2), SW2.1
- net at J1.1 (Pin_1): now also SW3.3 (A); no longer SW3.1 (B)
- net at SW2.2: now also U1.11 (GPIO18/D10/MOSI); no longer U1.8 (GPIO17/D7/RX)
- net at J2.1 (Pin_1), R1.2: now also SW3.1 (B); no longer SW3.2 (C)
Changed lines of the file:
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@@
+	)
+	(junction
+		(at 148.59 82.55)
+		(diameter 0)
+		(color 0 0 0 0)
 	)
 	(junction
@@
 	)
 	(junction
-		(at 107.95 77.47)
-		(diameter 0)
-		(color 0 0 0 0)
-	)
-	(junction
 		(at 180.34 111.76)
 		(diameter 0)
@@
 	)
 	(junction
-		(at 77.47 77.47)
-		(diameter 0)
-		(color 0 0 0 0)
-	)
-	(junction
 		(at 158.75 101.6)
 		(diameter 0)
@@
 	)
 	(junction
+		(at 77.47 82.55)
+		(diameter 0)
+		(color 0 0 0 0)
+	)
+	(junction
 		(at 120.65 64.77)
 		(diameter 0)
@@
 	)
 	(no_connect
-		(at 194.31 93.98)
+		(at 194.31 99.06)
 	)
 	(no_connect
@@
 	)
 	(no_connect
+		(at 147.32 116.84)
+	)
+	(no_connect
 		(at 147.32 109.22)
 	)
@@
 	)
 	(no_connect
-		(at 147.32 105.41)
-	)
-	(no_connect
 		(at 147.32 93.98)
 	)
@@
 	(wire
 		(pts
-			(xy 77.47 73.66) (xy 77.47 77.47)
+			(xy 77.47 73.66) (xy 77.47 82.55)
 		)
 		(stroke
@@
 	(wire
 		(pts
-			(xy 77.47 77.47) (xy 77.47 123.19)
+			(xy 184.15 96.52) (xy 182.88 96.52)
 		)
 		(stroke
@@
 	(wire
 		(pts
-			(xy 182.88 96.52) (xy 184.15 96.52)
-		)
-		(stroke
-			(width 0)
-			(type default)
-		)
-	)
-	(wire
-		(pts
 			(xy 167.64 101.6) (xy 175.26 101.6)
 		)
@@
 	(wire
 		(pts
+			(xy 182.88 96.52) (xy 182.88 109.22)
+		)
+		(stroke
+			(width 0)
+			(type default)
+		)
+	)
+	(wire
+		(pts
 			(xy 113.03 49.53) (xy 113.03 57.15)
 		)
@@
 	(wire
 		(pts
+			(xy 77.47 82.55) (xy 77.47 123.19)
+		)
+		(stroke
+			(width 0)
+			(type default)
+		)
+	)
+	(wire
+		(pts
 			(xy 90.17 109.22) (xy 97.79 109.22)
 		)
@@
 	(wire
 		(pts
-			(xy 147.32 123.19) (xy 147.32 116.84)
+			(xy 182.88 74.93) (xy 182.88 81.28)
 		)
 		(stroke
@@
 	(wire
 		(pts
+			(xy 149.86 123.19) (xy 149.86 105.41)
+		)
+		(stroke
+			(width 0)
+			(type default)
+		)
+	)
+	(wire
+		(pts
 			(xy 125.73 49.53) (xy 125.73 77.47)
 		)
@@
 	(wire
 		(pts
-			(xy 148.59 52.07) (xy 148.59 97.79)
-		)
-		(stroke
-			(width 0)
-			(type default)
-		)
-	)
-	(wire
-		(pts
-			(xy 182.88 102.87) (xy 182.88 109.22)
+			(xy 148.59 52.07) (xy 148.59 82.55)
 		)
 		(stroke
@@
 	(wire
 		(pts
-			(xy 182.88 74.93) (xy 182.88 96.52)
-		)
-		(stroke
-			(width 0)
-			(type default)
-		)
-	)
-	(wire
-		(pts
 			(xy 92.71 113.03) (xy 92.71 67.31)
 		)
@@
 	(wire
 		(pts
+			(xy 77.47 82.55) (xy 148.59 82.55)
+		)
+		(stroke
+			(width 0)
+			(type default)
+		)
+	)
+	(wire
+		(pts
 			(xy 161.29 100.33) (xy 161.29 101.6)
 		)
@@
 	(wire
 		(pts
-			(xy 194.31 99.06) (xy 194.31 102.87)
-		)
-		(stroke
-			(width 0)
-			(type default)
-		)
-	)
-	(wire
-		(pts
 			(xy 118.11 49.53) (xy 118.11 52.07)
 		)
@@
 	(wire
 		(pts
-			(xy 182.88 102.87) (xy 194.31 102.87)
-		)
-		(stroke
-			(width 0)
-			(type default)
-		)
-	)
-	(wire
-		(pts
-			(xy 87.63 123.19) (xy 147.32 123.19)
+			(xy 87.63 123.19) (xy 149.86 123.19)
 		)
 		(stroke
@@
 	(wire
 		(pts
+			(xy 194.31 81.28) (xy 194.31 93.98)
+		)
+		(stroke
+			(width 0)
+			(type default)
+		)
+	)
+	(wire
+		(pts
+			(xy 148.59 82.55) (xy 148.59 97.79)
+		)
+		(stroke
+			(width 0)
+			(type default)
+		)
+	)
+	(wire
+		(pts
 			(xy 157.48 97.79) (xy 154.94 97.79)
 		)
@@
 	(wire
 		(pts
+			(xy 147.32 105.41) (xy 149.86 105.41)
+		)
+		(stroke
+			(width 0)
+			(type default)
+		)
+	)
+	(wire
+		(pts
 			(xy 115.57 77.47) (xy 120.65 77.47)
 		)
@@
 	(wire
 		(pts
+			(xy 182.88 81.28) (xy 194.31 81.28)
+		)
+		(stroke
+			(width 0)
+			(type default)
+		)
+	)
+	(wire
+		(pts
 			(xy 115.57 49.53) (xy 115.57 77.47)
 		)
 		(stroke
-			(width 0)
-			(type default)
-		)
-	)
-	(wire
-		(pts
-			(xy 77.47 77.47) (xy 107.95 77.47)
-		)
-		(stroke

Commit message: Update 3D cases and pcb,hardware documentation
Parts:
- F1: footprint TestPoint:TestPoint_2Pads_Pitch2.54mm_Drill0.8mm -> Capacitor_THT:C_Disc_D4.3mm_W1.9mm_P5.00mm
Changed lines of the file:
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@@
 			)
 		)
-		(property "Footprint" "TestPoint:TestPoint_2Pads_Pitch2.54mm_Drill0.8mm"
+		(property "Footprint" "Capacitor_THT:C_Disc_D4.3mm_W1.9mm_P5.00mm"
 			(at 181.61 92.71 0)
 			(effects
